File: shy_bot_pcb/shy_bot_pcb.sch (KiCad schematic (older format))
At the start: 28 parts, among them J1 Barrel_Jack, J2 DB15_Female_HighDensity, J3 DB15_Male_HighDensity, J4 DB15_Male_HighDensity, Q1 MOSFET_N, U1 linear_servo_iris, U10 lin_servo_w_conn_X, U11 locking_servo_conn, U12 lin_servo_w_conn_Y, U13 locking_servo_conn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

Commit message: updated diagram
Parts:
- added R?: 10k, symbol R_Small
Connections:
- net labels added: UpBoard_to_Arduino_serial_GND, UpBoard_to_Arduino_serial_VCC
- wire segments 186 -> 195
- no-connect marks 75 -> 71
Other:
- moved on the sheet: J2, J3, U4, U5, U6, U7
