File: PCB_V2/JoelHobbieRobots.sch (KiCad schematic (older format))
At the start: 10 parts, among them J1 Conn_02x20_Odd_Even, J2 Barrel_Jack, J3 DB15_Female_HighDensity, J4 Conn_01x08, J5 Conn_01x04, J6 Conn_01x08, J7 Conn_01x08, Q1 MOSFET-N

Commit message: Corrected errors andwarnings. If any warning appear, disregard them.
Parts:
- J1: value Conn_02x20_Odd_Even -> UpBoard 2x20
- J3: value DB15_Female_HighDensity -> DSub_Out
- J4: value Conn_01x08 -> H-Bridge_3; footprint (none) -> Pin_Headers:Pin_Header_Straight_1x08_Pitch2.54mm; Field10 (none) -> DIR; Field11 (none) -> GND; Field4 (none) -> V+; Field5 (none) -> 5V(out); Field6 (none) -> FF2; Field7 (none) -> FF1; Field8 (none) -> RESET; Field9 (none) -> PWM
- J5: Field4 (none) -> Vin(12V); Field5 (none) -> GND; Field6 (none) -> GND; Field7 (none) -> Out(5V)
- J6: value Conn_01x08 -> H-Bridge_2; footprint (none) -> Pin_Headers:Pin_Header_Straight_1x08_Pitch2.54mm; Field10 (none) -> DIR; Field11 (none) -> GND; Field4 (none) -> V+; Field5 (none) -> 5V(out); Field6 (none) -> FF2; Field7 (none) -> FF1; Field8 (none) -> RESET; Field9 (none) -> PWM
- J7: value Conn_01x08 -> H-Bridge_1; footprint (none) -> Pin_Headers:Pin_Header_Straight_1x08_Pitch2.54mm; Field10 (none) -> DIR; Field11 (none) -> GND; Field4 (none) -> V+; Field5 (none) -> 5V(out); Field6 (none) -> FF2; Field7 (none) -> FF1; Field8 (none) -> RESET; Field9 (none) -> PWM
- Q1: footprint Pin_Headers:Pin_Header_Straight_1x03_Pitch2.54mm -> TO_SOT_Packages_SMD:SOT-23_Handsoldering
Changed lines of the file:
@@
 encoding utf-8
 Sheet 1 1
-Title "Joel Hobbie's Robots"
+Title "Shy Bot"
 Date ""
 Rev "V1.0"
@@
 P 1450 3150
 F 0 "J1" H 1500 4150 50  0000 C CNN
-F 1 "Conn_02x20_Odd_Even" H 1500 2050 50  0000 C CNN
+F 1 "UpBoard 2x20" H 1500 2050 50  0000 C CNN
 F 2 "Pin_Headers:Pin_Header_Straight_2x20_Pitch2.54mm" H 1450 3150 50  0001 C CNN
 F 3 "" H 1450 3150 50  0001 C CNN
@@
 F 0 "Q1" H 3900 3675 45  0000 L BNN
 F 1 "MOSFET-N" H 3900 3600 45  0000 L BNN
-F 2 "Pin_Headers:Pin_Header_Straight_1x03_Pitch2.54mm" H 3700 3650 60  0001 C CNN
+F 2 "TO_SOT_Packages_SMD:SOT-23_Handsoldering" H 3700 3650 60  0001 C CNN
 F 3 "" H 3700 3650 60  0001 C CNN
 	1    3700 3650
@@
 P 9800 2050
 F 0 "J3" H 9800 2900 50  0000 C CNN
-F 1 "DB15_Female_HighDensity" H 9800 2800 50  0000 C CNN
+F 1 "DSub_Out" H 9800 2800 50  0000 C CNN
 F 2 "Connectors_DSub:DSUB-15-HD_Female_Horizontal_Pitch2.29x1.98mm_EdgePinOffset8.35mm_Housed_MountingHolesOffset10.89mm" H 8850 2450 50  0001 C CNN
 F 3 "" H 8850 2450 50  0001 C CNN
@@
 $EndComp
 $Comp
-L +5V #PWR06
-U 1 1 5B83171E
-P 7250 3250
-F 0 "#PWR06" H 7250 3100 50  0001 C CNN
-F 1 "+5V" H 7250 3390 50  0000 C CNN
-F 2 "" H 7250 3250 50  0001 C CNN
-F 3 "" H 7250 3250 50  0001 C CNN
-	1    7250 3250
-	1    0    0    -1
-$EndComp
-$Comp
-L +12V #PWR07
+L +12V #PWR06
 U 1 1 5B8317DE
 P 5300 1600
-F 0 "#PWR07" H 5300 1450 50  0001 C CNN
+F 0 "#PWR06" H 5300 1450 50  0001 C CNN
 F 1 "+12V" H 5300 1740 50  0000 C CNN
 F 2 "" H 5300 1600 50  0001 C CNN
@@
 drive_sig_X
 $Comp
-L +12V #PWR08
+L +12V #PWR07
 U 1 1 5B831E56
 P 9050 1200
-F 0 "#PWR08" H 9050 1050 50  0001 C CNN
+F 0 "#PWR07" H 9050 1050 50  0001 C CNN
 F 1 "+12V" H 9050 1340 50  0000 C CNN
 F 2 "" H 9050 1200 50  0001 C CNN
@@
 $EndComp
 $Comp
-L +5V #PWR09
+L +5V #PWR08
 U 1 1 5B832536
 P 1950 2100
-F 0 "#PWR09" H 1950 1950 50  0001 C CNN
+F 0 "#PWR08" H 1950 1950 50  0001 C CNN
 F 1 "+5V" H 1950 2240 50  0000 C CNN
 F 2 "" H 1950 2100 50  0001 C CNN
@@
 $EndComp
 $Comp
-L GND #PWR010
+L GND #PWR09
 U 1 1 5B832553
 P 2100 2500
-F 0 "#PWR010" H 2100 2250 50  0001 C CNN
+F 0 "#PWR09" H 2100 2250 50  0001 C CNN
 F 1 "GND" H 2100 2350 50  0000 C CNN
 F 2 "" H 2100 2500 50  0001 C CNN
@@
 $EndComp
 $Comp
-L GND #PWR011
+L GND #PWR010
 U 1 1 5B832612
 P 950 2700
-F 0 "#PWR011" H 950 2450 50  0001 C CNN
+F 0 "#PWR010" H 950 2450 50  0001 C CNN
 F 1 "GND" H 950 2550 50  0000 C CNN
 F 2 "" H 950 2700 50  0001 C CNN
@@
 F 2 "Pin_Headers:Pin_Header_Straight_1x04_Pitch2.54mm" H 9950 4550 50  0001 C CNN
 F 3 "" H 9950 4550 50  0001 C CNN
+F 4 "Vin(12V)" H 9650 4400 60  0000 C CNN "Field4"
+F 5 "GND" H 9700 4500 60  0000 C CNN "Field5"
+F 6 "GND" H 9700 4600 60  0000 C CNN "Field6"
+F 7 "Out(5V)" H 9650 4700 60  0000 C CNN "Field7"
 	1    9950 4550
 	1    0    0    -1
@@
 P 1000 5300
 F 0 "J4" H 1000 5700 50  0000 C CNN
-F 1 "Conn_01x08" H 1000 4800 50  0000 C CNN
-F 2 "" H 1000 5300 50  0001 C CNN
+F 1 "H-Bridge_3" H 1000 4800 50  0000 C CNN
+F 2 "Pin_Headers:Pin_Header_Straight_1x08_Pitch2.54mm" H 1000 5300 50  0001 C CNN
 F 3 "" H 1000 5300 50  0001 C CNN
+F 4 "V+" H 700 5550 60  0000 C CNN "Field4"
+F 5 "5V(out)" H 650 5450 60  0000 C CNN "Field5"
+F 6 "FF2" H 700 5350 60  0000 C CNN "Field6"
+F 7 "FF1" H 700 5250 60  0000 C CNN "Field7"
+F 8 "RESET" H 700 5150 60  0000 C CNN "Field8"
+F 9 "PWM" H 700 5050 60  0000 C CNN "Field9"
+F 10 "DIR" H 700 4950 60  0000 C CNN "Field10"
+F 11 "GND" H 700 4850 60  0000 C CNN "Field11"
 	1    1000 5300
 	-1   0    0    1
@@
 P 1000 6350
 F 0 "J6" H 1000 6750 50  0000 C CNN
-F 1 "Conn_01x08" H 1000 5850 50  0000 C CNN
-F 2 "" H 1000 6350 50  0001 C CNN
+F 1 "H-Bridge_2" H 1000 5850 50  0000 C CNN
+F 2 "Pin_Headers:Pin_Header_Straight_1x08_Pitch2.54mm" H 1000 6350 50  0001 C CNN
 F 3 "" H 1000 6350 50  0001 C CNN
+F 4 "V+" H 750 6600 60  0000 C CNN "Field4"
+F 5 "5V(out)" H 650 6500 60  0000 C CNN "Field5"
+F 6 "FF2" H 700 6400 60  0000 C CNN "Field6"
+F 7 "FF1" H 700 6300 60  0000 C CNN "Field7"
+F 8 "RESET" H 700 6200 60  0000 C CNN "Field8"
+F 9 "PWM" H 700 6100 60  0000 C CNN "Field9"
+F 10 "DIR" H 700 6000 60  0000 C CNN "Field10"
+F 11 "GND" H 700 5900 60  0000 C CNN "Field11"
 	1    1000 6350
 	-1   0    0    1
@@
 P 1000 7350
 F 0 "J7" H 1000 7750 50  0000 C CNN
-F 1 "Conn_01x08" H 1000 6850 50  0000 C CNN
-F 2 "" H 1000 7350 50  0001 C CNN
+F 1 "H-Bridge_1" H 1000 6850 50  0000 C CNN
+F 2 "Pin_Headers:Pin_Header_Straight_1x08_Pitch2.54mm" H 1000 7350 50  0001 C CNN
 F 3 "" H 1000 7350 50  0001 C CNN
+F 4 "V+" H 750 7600 60  0000 C CNN "Field4"
+F 5 "5V(out)" H 650 7500 60  0000 C CNN "Field5"
+F 6 "FF2" H 750 7400 60  0000 C CNN "Field6"
+F 7 "FF1" H 750 7300 60  0000 C CNN "Field7"
+F 8 "RESET" H 700 7200 60  0000 C CNN "Field8"
+F 9 "PWM" H 700 7100 60  0000 C CNN "Field9"
+F 10 "DIR" H 700 7000 60  0000 C CNN "Field10"
+F 11 "GND" H 700 6900 60  0000 C CNN "Field11"
 	1    1000 7350
 	-1   0    0    1
 $EndComp
 $Comp
-L +5V #PWR012
+L +5V #PWR011
 U 1 1 5B856293
 P 8800 1200
-F 0 "#PWR012" H 8800 1050 50  0001 C CNN
+F 0 "#PWR011" H 8800 1050 50  0001 C CNN
 F 1 "+5V" H 8800 1340 50  0000 C CNN
 F 2 "" H 8800 1200 50  0001 C CNN
@@
 drive_sig_W
 $Comp
-L +5V #PWR013
+L +5V #PWR012
 U 1 1 5B85AE28
 P 1800 5600
-F 0 "#PWR013" H 1800 5450 50  0001 C CNN
+F 0 "#PWR012" H 1800 5450 50  0001 C CNN
 F 1 "+5V" H 1800 5740 50  0000 C CNN
 F 2 "" H 1800 5600 50  0001 C CNN
@@
 $EndComp
 $Comp
-L +5V #PWR014
+L +5V #PWR013
 U 1 1 5B85AE51
 P 1750 7650
-F 0 "#PWR014" H 1750 7500 50  0001 C CNN
+F 0 "#PWR013" H 1750 7500 50  0001 C CNN
 F 1 "+5V" H 1750 7790 50  0000 C CNN
 F 2 "" H 1750 7650 50  0001 C CNN
@@
 $EndComp
 $Comp
-L +5V #PWR015
+L +5V #PWR014
 U 1 1 5B85AE7A
 P 1800 6600
-F 0 "#PWR015" H 1800 6450 50  0001 C CNN
+F 0 "#PWR014" H 1800 6450 50  0001 C CNN
 F 1 "+5V" H 1800 6740 50  0000 C CNN
 F 2 "" H 1800 6600 50  0001 C CNN
@@
 D5
 $Comp
-L GND #PWR016
+L GND #PWR015
 U 1 1 5B85BC0A
 P 2200 4850
-F 0 "#PWR016" H 2200 4600 50  0001 C CNN
+F 0 "#PWR015" H 2200 4600 50  0001 C CNN
 F 1 "GND" H 2200 4700 50  0000 C CNN
 F 2 "" H 2200 4850 50  0001 C CNN
@@
 $EndComp
 $Comp
-L GND #PWR017
+L GND #PWR016
 U 1 1 5B85BC33
 P 2100 5900
-F 0 "#PWR017" H 2100 5650 50  0001 C CNN
+F 0 "#PWR016" H 2100 5650 50  0001 C CNN
 F 1 "GND" H 2100 5750 50  0000 C CNN
 F 2 "" H 2100 5900 50  0001 C CNN
@@
 $EndComp
 $Comp
-L GND #PWR018
+L GND #PWR017
 U 1 1 5B85BC5C
 P 2050 6900
-F 0 "#PWR018" H 2050 6650 50  0001 C CNN
+F 0 "#PWR017" H 2050 6650 50  0001 C CNN
 F 1 "GND" H 2050 6750 50  0000 C CNN
 F 2 "" H 2050 6900 50  0001 C CNN
@@
 NoConn ~ 5850 3050
 $Comp
-L GND #PWR019
+L GND #PWR018
 U 1 1 5B85CC67
 P 7800 3050
-F 0 "#PWR019" H 7800 2800 50  0001 C CNN
+F 0 "#PWR018" H 7800 2800 50  0001 C CNN
 F 1 "GND" H 7800 2900 50  0000 C CNN
 F 2 "" H 7800 3050 50  0001 C CNN
@@
 $EndComp
 $Comp
-L PWR_FLAG #FLG020
+L PWR_FLAG #FLG019
 U 1 1 5B86B8BC
-P 5600 1350
-F 0 "#FLG020" H 5600 1425 50  0001 C CNN
-F 1 "PWR_FLAG" H 5600 1500 50  0000 C CNN
-F 2 "" H 5600 1350 50  0001 C CNN
-F 3 "" H 5600 1350 50  0001 C CNN
-	1    5600 1350
-	1    0    0    -1
-$EndComp
-$Comp
-L PWR_FLAG #FLG021
-U 1 1 5B86BD0A
-P 4550 1550
-F 0 "#FLG021" H 4550 1625 50  0001 C CNN
-F 1 "PWR_FLAG" H 4550 1700 50  0000 C CNN
-F 2 "" H 4550 1550 50  0001 C CNN
-F 3 "" H 4550 1550 50  0001 C CNN
-	1    4550 1550
-	-1   0    0    1
-$EndComp
-$Comp
-L GND #PWR022
+P 4600 1500
+F 0 "#FLG019" H 4600 1575 50  0001 C CNN
+F 1 "PWR_FLAG" H 4600 1650 50  0000 C CNN
+F 2 "" H 4600 1500 50  0001 C CNN
+F 3 "" H 4600 1500 50  0001 C CNN
+	1    4600 1500
+	1    0    0    -1
+$EndComp
+$Comp
+L GND #PWR020
 U 1 1 5B86C2E4
 P 3800 3250
-F 0 "#PWR022" H 3800 3000 50  0001 C CNN
+F 0 "#PWR020" H 3800 3000 50  0001 C CNN
 F 1 "GND" H 3800 3100 50  0000 C CNN
 F 2 "" H 3800 3250 50  0001 C CNN
@@
 Connection ~ 9650 4650
 Wire Wire Line
-	7250 3250 7050 3250
-Wire Wire Line
 	5100 1350 5100 1600
 Wire Wire Line
@@
 	7050 3050 7800 3050
 Wire Wire Line
-	4550 1500 4900 1500
-Connection ~ 4900 1500
-Wire Wire Line
-	4550 1500 4550 1550
-Wire Wire Line
-	5100 1400 5600 1400
-Wire Wire Line
-	5600 1400 5600 1350
-Connection ~ 5100 1400
-Wire Wire Line
 	3600 4100 3450 4100
 Wire Wire Line
@@
 Connection ~ 3600 3400
 $Comp
-L GND #PWR023
+L GND #PWR021
 U 1 1 5B86C7C6
 P 4500 3150
-F 0 "#PWR023" H 4500 2900 50  0001 C CNN
+F 0 "#PWR021" H 4500 2900 50  0001 C CNN
 F 1 "GND" H 4500 3000 50  0000 C CNN
 F 2 "" H 4500 3150 50  0001 C CNN
@@
 Wire Wire Line
 	5300 3250 5850 3250
+$Comp
+L +5V #PWR022
+U 1 1 5B880A48
+P 7300 3250
+F 0 "#PWR022" H 7300 3100 50  0001 C CNN
+F 1 "+5V" H 7300 3390 50  0000 C CNN
+F 2 "" H 7300 3250 50  0001 C CNN
+F 3 "" H 7300 3250 50  0001 C CNN
+	1    7300 3250
+	1    0    0    -1
+$EndComp
+Wire Wire Line
+	7050 3250 7300 3250
+$Comp
+L PWR_FLAG #FLG023
+U 1 1 5B86BD0A
+P 5250 1700
+F 0 "#FLG023" H 5250 1775 50  0001 C CNN
+F 1 "PWR_FLAG" H 5250 1850 50  0000 C CNN
+F 2 "" H 5250 1700 50  0001 C CNN
+F 3 "" H 5250 1700 50  0001 C CNN
+	1    5250 1700
+	-1   0    0    1
+$EndComp
+Wire Wire Line
+	4600 1500 4900 1500
+Connection ~ 4900 1500
+Wire Wire Line
+	5250 1700 5250 1600
+Connection ~ 5250 1600
 $EndSCHEMATC
